Commit message: правки murom_description для работы в rviz

File: murom/murom_description/urdf/kinect/kinect.urdf.xacro (robot description, xacro)
@@ -27,5 +27,5 @@
        <origin xyz="0 0 0" rpy="0 0 ${M_PI/2}"/>
         <geometry>
-         <mesh filename="package://turtlebot_description/meshes/sensors/kinect.dae"/>
+         <mesh filename="package://murom_description/meshes/kinect.dae"/>
         </geometry>
       </visual>
@@ -60,5 +60,5 @@
 	<link name="camera_depth_optical_frame"/>
 	<!-- Kinect sensor for simulation -->
-	<turtlebot_sim_3dsensor/>
+	<murom_sim_3dsensor/>
   </xacro:macro>
 </robot>

File: murom/murom_description/urdf/murom.urdf.xacro (robot description, xacro)
@@ -104,6 +104,6 @@
   </link>
   <joint
-    name="spj"
-    type="fixed">
+    name="Park_move"
+    type="continuous">
     <origin
       xyz="-0.35647938563719 -0.00728806900000959 -0.278593729468106"
@@ -115,4 +115,6 @@
     <axis
       xyz="0 -1 0" />
+<limit effort="1000" velocity="10"/>
+   <dynamics damping="0.7" friction="0.1"/>
   </joint>
   <link
@@ -158,5 +160,5 @@
   <joint
     name="wheel_left_joint"
-    type="fixed">
+    type="continuous">
     <origin
       xyz="0.0368499999999981 0.267211930999997 -0.127248471181616"
@@ -168,4 +170,6 @@
     <axis
       xyz="0 -1 0" />
+<limit effort="1000" velocity="10"/>
+   <dynamics damping="0.7" friction="0.1"/>
   </joint>
   <link
@@ -211,5 +215,5 @@
   <joint
     name="wheel_right_joint"
-    type="fixed">
+    type="continuous">
     <origin
       xyz="0.0368500000000074 -0.266788069000003 -0.127248471181616"
@@ -221,4 +225,6 @@
     <axis
       xyz="0 1 0" />
+<limit effort="1000" velocity="10"/>
+   <dynamics damping="0.7" friction="0.1"/>
   </joint>
   <link
@@ -263,6 +269,6 @@
   </link>
   <joint
-    name="pj"
-    type="fixed">
+    name="Trunk_rotate"
+    type="revolute">
     <origin
       xyz="0 0 0.310000000000001"
@@ -274,6 +280,6 @@
     <axis
       xyz="0 0 1" />
-<limit effort="1000" velocity="1000"/>
-   <dynamics damping="0.7" friction="0.0"/>
+<limit effort="1000" velocity="10" lower="${-M_PI/2}" upper="${M_PI/2}"/>
+   <dynamics damping="0.7" friction="0.1"/>
   </joint>
   <link
@@ -318,6 +324,6 @@
   </link>
   <joint
-    name="tdj"
-    type="fixed">
+    name="Belly_turn"
+    type="revolute">
     <origin
       xyz="-0.0545323092339866 0.113440016086032 0.148599999999998"
@@ -329,4 +335,6 @@
     <axis
       xyz="0 1 0" />
+<limit effort="1000" velocity="10" lower="0" upper="${M_PI/2}"/>
+   <dynamics damping="0.7" friction="0.1"/>
   </joint>
   <link
@@ -371,6 +379,6 @@
   </link>
   <joint
-    name="tuj"
-    type="fixed">
+    name="Spine_move"
+    type="revolute">
     <origin
       xyz="-0.0613353782819227 -0.178500000000035 0.371988556686935"
@@ -382,4 +390,6 @@
     <axis
       xyz="0 -1 0" />
+<limit effort="1000" velocity="10" lower="${-M_PI/4}" upper="${4*M_PI/5}"/>
+   <dynamics damping="0.7" friction="0.1"/>
   </joint>
   <link
@@ -424,6 +434,6 @@
   </link>
   <joint
-    name="nj"
-    type="fixed">
+    name="Neck_move"
+    type="revolute">
     <origin
       xyz="-0.0516500646336157 0.093000000000035 0.325629296136459"
@@ -435,4 +445,6 @@
     <axis
       xyz="0 1 0" />
+<limit effort="1000" velocity="10" lower="0" upper="${M_PI/2}"/>
+   <dynamics damping="0.7" friction="0.1"/>
   </joint>
   <link
@@ -477,6 +489,6 @@
   </link>
   <joint
-    name="hj"
-    type="fixed">
+    name="Head_rotate"
+    type="revolute">
     <origin
       xyz="-0.0176086934682474 -0.0120000000000006 0.106554839938601"
@@ -488,4 +500,6 @@
     <axis
       xyz="0 0 1" />
+<limit effort="1000" velocity="10" lower="${-M_PI/2}" upper="${M_PI/2}"/>
+   <dynamics damping="0.7" friction="0.1"/>
   </joint>
   <sensor_kinect  parent="base_link"/>

Commit message: правки для gh

File: murom/murom_description/urdf/kinect/kinect.urdf.xacro (robot description, xacro)
@@ -1,5 +1,5 @@
 <?xml version="1.0"?>
 <robot name="sensor_kinect" xmlns:xacro="http://ros.org/wiki/xacro">
-<!--  <xacro:include filename="$(find murom_description)/urdf/turtlebot_gazebo.urdf.xacro"/>-->
+  <xacro:include filename="$(find murom_description)/urdf/murom_gazebo.urdf.xacro"/>
   <xacro:include filename="$(find murom_description)/urdf/murom_properties.urdf.xacro"/>
   <xacro:property name="kinect_cam_py" value="-0.0125"/>
@@ -7,5 +7,5 @@
   <xacro:macro name="sensor_kinect" params="parent">
     <joint name="camera_rgb_joint" type="fixed">
-      <origin xyz="${cam_px} ${kinect_cam_py} ${cam_pz}" rpy="${cam_or} ${cam_op} ${cam_oy}"/>
+      <origin xyz="${cam_px} ${kinect_cam_py} ${cam_pz}" rpy="${cam_or} 0.26 ${cam_oy}"/>
       <parent link="${parent}"/>
       <child link="camera_rgb_frame" />

File: murom/murom_description/urdf/murom.urdf.xacro (robot description, xacro)
@@ -1,20 +1,46 @@
 <?xml version="1.0"?>
 <robot name="murom" xmlns:xacro="http://ros.org/wiki/xacro">
-  <xacro:include filename="$(find murom_description)/urdf/kinect/kinect.urdf.xacro"/>
+  <xacro:include filename="$(find murom_description)/urdf/kinect/kinect2.urdf.xacro"/>
   <xacro:include filename="$(find murom_description)/urdf/common_properties.urdf.xacro"/>
   <xacro:include filename="$(find murom_description)/urdf/murom_properties.urdf.xacro"/>
+  <xacro:include filename="$(find murom_description)/urdf/wheel.urdf.xacro" />
   <!-- ros_control plugin -->
-  <gazebo>
+<!-- <gazebo>
     <plugin name="gazebo_ros_control" filename="libgazebo_ros_control.so">
       <robotNamespace>/murom</robotNamespace>
     </plugin>
   </gazebo>
+   <gazebo>
+    <plugin name="differential_drive_controller" filename="libgazebo_ros_diff_drive.so">
+      <rosDebugLevel>Debug</rosDebugLevel>
+      <publishWheelTF>false</publishWheelTF>
+      <robotNamespace>/</robotNamespace>
+      <publishTf>1</publishTf>
+      <publishWheelJointState>false</publishWheelJointState>
+      <alwaysOn>true</alwaysOn>
+      <updateRate>50.0</updateRate>
+      <leftJoint>wheel_left_joint</leftJoint>
+      <rightJoint>wheel_right_joint</rightJoint>
+      <wheelSeparation>0.5</wheelSeparation>
+      <wheelDiameter>0.3</wheelDiameter>
+      <broadcastTF>1</broadcastTF>
+      <wheelTorque>50</wheelTorque>
+      <wheelAcceleration>1.8</wheelAcceleration>
+      <commandTopic>cmd_vel</commandTopic>
+      <enableOdometryTF>false</enableOdometryTF>
+      <odometryFrame>odom</odometryFrame>
+      <odometryTopic>odom</odometryTopic>
+      <robotBaseFrame>base_footprint</robotBaseFrame>
+    </plugin>
+  </gazebo>
+-->
 <link
-    name="base_footprint"/>
+    name="base_footprint">
+</link>
   <joint
     name="base_joint"
     type="fixed">
     <origin
-      xyz="0 0 0.3"
+      xyz="0 0 0.4"
       rpy="0 0 0" />
     <parent
@@ -26,17 +52,17 @@
     name="base_link">
     <inertial>
-      <origin
-        xyz="-0.00558505045857072 0.000223008604259885 0.0390613117723667"
-        rpy="0 0 0" />
-      <mass
-        value="43.2053004192762" />
-      <inertia
-        ixx="2.65958282143013"
-        ixy="0.000274170236096077"
-        ixz="0.0713810073451908"
-        iyy="2.52723505537043"
-        iyz="9.21060215788137E-05"
-        izz="3.15073786919698" />
-    </inertial>
+         <origin
+           xyz="0.028634 -0.017991 0.021937"
+           rpy="0 0 0" />
+         <mass
+           value="72.98" />
+         <inertia
+           ixx="4.9013"
+           ixy="0.0071913"
+           ixz="-0.00020072"
+           iyy="4.3205"
+           iyz="-0.056159"
+           izz="6.1094" />
+       </inertial>
     <visual>
       <origin
@@ -53,5 +79,11 @@
       </material>
     </visual>
-    <collision>
+ <collision>
+        <origin xyz="0.0 0.0 0.05" rpy="0 0 0"/>
+  	    <geometry>
+  	      <box size="0.5 0.5 0.5"/>
+  	    </geometry>
+  	  </collision>
+<!--    <collision>
       <origin
         xyz="0 0 0"
@@ -61,26 +93,26 @@
           filename="package://murom_description/meshes/found.STL" />
       </geometry>
-    </collision>
-  </link>
-  <link
+    </collision>-->
+  </link>
+<!--  <link
     name="supwheel">
     <inertial>
+          <origin
+            xyz="0.027714 -0.014703 0.01016"
+            rpy="0 0 0" />
+          <mass
+            value="0.086014" />
+          <inertia
+            ixx="0.00026204"
+            ixy="2.3732E-06"
+            ixz="1.3983E-05"
+            iyy="0.00027128"
+            iyz="4.307E-05"
+            izz="3.1939E-05" />
+        </inertial>
+    <visual>
       <origin
         xyz="-3.48054918219987E-14 0.01 8.49877695996426E-09"
         rpy="0 0 0" />
-      <mass
-        value="0.252410366826367" />
-      <inertia
-        ixx="4.22011549053702E-05"
-        ixy="5.0719450726252E-12"
-        ixz="-5.10991065078981E-21"
-        iyy="7.03711150556965E-05"
-        iyz="-2.30990289511718E-20"
-        izz="4.22013245287302E-05" />
-    </inertial>
-    <visual>
-      <origin
-        xyz="0 0 0"
-        rpy="0 0 0" />
       <geometry>
         <mesh
@@ -95,5 +127,5 @@
     <collision>
       <origin
-        xyz="0 0 0"
+        xyz="-3.48054918219987E-14 0.01 8.49877695996426E-09"
         rpy="0 0 0" />
       <geometry>
@@ -105,5 +137,5 @@
   <joint
     name="Park_move"
-    type="continuous">
+    type="fixed">
     <origin
       xyz="-0.35647938563719 -0.00728806900000959 -0.278593729468106"
@@ -114,24 +146,63 @@
       link="supwheel" />
     <axis
-      xyz="0 -1 0" />
-<limit effort="1000" velocity="10"/>
-   <dynamics damping="0.7" friction="0.1"/>
-  </joint>
-  <link
+      xyz="0.02 0  0.01" />
+<limit effort="300" velocity="10"/>
+   <dynamics damping="0.0" friction="0.0"/>
+  </joint>
+ <gazebo reference="supwheel">
+    <turnGravityOff>false</turnGravityOff>
+  </gazebo>
+-->
+ <property name="caster_b_height" value="0.04" />
+  <property name="caster_b_radius" value="0.025" />
+  <property name="caster_b_mass" value="0.5" /> <!-- in kg-->
+    <link name="caster_back_link">
+    <visual>
+      <origin xyz="0.02 0.02 0 " rpy="${M_PI/2} 0 0" />
+      <geometry>
+	<sphere radius="${caster_b_radius}" />
+      </geometry>
+      <material name="Black" />
+    </visual>
+      <collision>
+        <geometry>
+		<sphere radius="${caster_b_radius}" />
+        </geometry>
+      <origin xyz="0 0.02 0 " rpy="${M_PI/2} 0 0" />
+      </collision>
+      <inertial>
+        <mass value="${caster_b_mass}" />
+        <origin xyz="0 0 0" />
+        <inertia ixx="0.001" ixy="0.0" ixz="0.0"
+                 iyy="0.001" iyz="0.0"
+                 izz="0.001" />
+      </inertial>
+    </link>
+    <joint name="caster_back_joint" type="fixed">
+      <parent link="base_link"/>
+      <child link="caster_back_link"/>
+      <origin xyz="-0.435 0.0 -0.25" rpy="${-M_PI/2} 0 0"/>
+    </joint>
+  <gazebo reference="caster_back_link">
+    <turnGravityOff>false</turnGravityOff>
+  </gazebo>
+  <wheel lr="right" parent="base_link" translateX="0.15" translateY="0.5" flipY="1"/>
+  <wheel lr="left" parent="base_link" translateX="0.15" translateY="-0.5" flipY="1"/>
+<!--  <link
     name="wheel_left_link">
     <inertial>
-      <origin
-        xyz="-1.08636716456001E-07 -0.0400666405449752 -1.45598615525211E-07"
-        rpy="0 0 0" />
-      <mass
-        value="38.5016876202174" />
-      <inertia
-        ixx="0.281294106347389"
-        ixy="3.70269664395719E-07"
-        ixz="-2.03741583151806E-06"
-        iyy="0.541042482295194"
-        iyz="-2.55348177673329E-07"
-        izz="0.281291684801198" />
-    </inertial>
+        <origin
+          xyz="0 0 0"
+          rpy="0 0 0" />
+        <mass
+          value="38.502" />
+        <inertia
+          ixx="0.28129"
+          ixy="2.1343E-06"
+          ixz="-4.4702E-07"
+          iyy="0.28129"
+          iyz="-4.9709E-08"
+          izz="0.54104" />
+      </inertial>
     <visual>
       <origin
@@ -169,24 +240,22 @@
       link="wheel_left_link" />
     <axis
-      xyz="0 -1 0" />
-<limit effort="1000" velocity="10"/>
-   <dynamics damping="0.7" friction="0.1"/>
+      xyz="0 1 0" />
   </joint>
   <link
     name="wheel_right_link">
     <inertial>
-      <origin
-        xyz="0.00400007774006554 0.040066489008572 -1.77615343599502E-07"
-        rpy="0 0 0" />
-      <mass
-        value="38.5015659404429" />
-      <inertia
-        ixx="0.281292585109412"
-        ixy="4.20506342151003E-07"
-        ixz="2.35864084102445E-06"
-        iyy="0.541041874307209"
-        iyz="1.55988542073103E-07"
-        izz="0.281292121004341" />
-    </inertial>
+         <origin
+           xyz="0 0 0"
+           rpy="0 0 0" />
+         <mass
+           value="38.502" />
+         <inertia
+           ixx="0.28129"
+           ixy="2.1343E-06"
+           ixz="-4.4703E-07"
+           iyy="0.28129"
+           iyz="-3.6422E-08"
+           izz="0.54104" />
+       </inertial>
     <visual>
       <origin
@@ -225,7 +294,5 @@
     <axis
       xyz="0 1 0" />
-<limit effort="1000" velocity="10"/>
-   <dynamics damping="0.7" friction="0.1"/>
-  </joint>
+  </joint>-->
   <link
     name="pillar">
@@ -237,10 +304,10 @@
         value="0.0531161397704353" />
       <inertia
-        ixx="1.7621925188156E-05"
-        ixy="-3.41800335229115E-06"
-        ixz="1.92231181336778E-11"
-        iyy="3.09757385697677E-05"
-        iyz="1.44724593440625E-10"
-        izz="1.67970057163936E-05" />
+        ixx="0.001"
+        ixy="0"
+        ixz="0"
+        iyy="0.001"
+        iyz="0"
+        izz="0.001" />
     </inertial>
     <visual>
@@ -270,5 +337,5 @@
   <joint
     name="Trunk_rotate"
-    type="revolute">
+    type="fixed">
     <origin
       xyz="0 0 0.310000000000001"
@@ -280,6 +347,6 @@
     <axis
       xyz="0 0 1" />
-<limit effort="1000" velocity="10" lower="${-M_PI/2}" upper="${M_PI/2}"/>
-   <dynamics damping="0.7" friction="0.1"/>
+<limit effort="300" velocity="1" lower="${-M_PI/2}" upper="${M_PI/2}"/>
+   <dynamics damping="50" friction="1"/>
   </joint>
   <link
@@ -290,12 +357,12 @@
         rpy="0 0 0" />
       <mass
-        value="2.43455936674416" />
+        value="10" />
       <inertia
-        ixx="0.0391766067371756"
-        ixy="1.35297180546079E-06"
-        ixz="-0.00173803195173356"
-        iyy="0.0205503137157225"
-        iyz="-2.79544515525284E-05"
-        izz="0.0193471460246358" />
+        ixx="0.03"
+        ixy="0"
+        ixz="0"
+        iyy="0.02"
+        iyz="0"
+        izz="0.02" />
     </inertial>
     <visual>
@@ -325,5 +392,5 @@
   <joint
     name="Belly_turn"
-    type="revolute">
+    type="fixed">
     <origin
       xyz="-0.0545323092339866 0.113440016086032 0.148599999999998"
@@ -335,6 +402,6 @@
     <axis
       xyz="0 1 0" />
-<limit effort="1000" velocity="10" lower="0" upper="${M_PI/2}"/>
-   <dynamics damping="0.7" friction="0.1"/>
+<limit effort="300" velocity="1" lower="0" upper="${M_PI/2}"/>
+   <dynamics damping="50" friction="1"/>
   </joint>
   <link
@@ -345,12 +412,12 @@
         rpy="0 0 0" />
       <mass
-        value="3.9054747412393" />
+        value="10" />
       <inertia
-        ixx="0.0780594086603757"
-        ixy="6.01331218089826E-05"
-        ixz="-0.00919269267657588"
-        iyy="0.0388143695460778"
-        iyz="-0.000187292947851412"
-        izz="0.0445355367000355" />
+        ixx="0.08"
+        ixy="0"
+        ixz="0"
+        iyy="0.04"
+        iyz="0"
+        izz="0.04" />
     </inertial>
     <visual>
@@ -380,5 +447,5 @@
   <joint
     name="Spine_move"
-    type="revolute">
+    type="fixed">
     <origin
       xyz="-0.0613353782819227 -0.178500000000035 0.371988556686935"
@@ -390,6 +457,6 @@
     <axis
       xyz="0 -1 0" />
-<limit effort="1000" velocity="10" lower="${-M_PI/4}" upper="${4*M_PI/5}"/>
-   <dynamics damping="0.7" friction="0.1"/>
+<limit effort="300" velocity="1" lower="${-M_PI/4}" upper="${4*M_PI/5}"/>
+   <dynamics damping="50" friction="1"/>
   </joint>
   <link
@@ -400,12 +467,12 @@
         rpy="0 0 0" />
       <mass
-        value="0.4503224240065" />
+        value="1" />
       <inertia
-        ixx="0.000219493904356614"
-        ixy="-2.3782519126248E-13"
-        ixz="-1.1935388635364E-05"
-        iyy="0.000214451258670037"
-        iyz="2.42313107702396E-12"
-        izz="0.000149242043540864" />
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